File: cad/pan_tilt_lidar.sch (EAGLE design)
At the start: 9 parts

Commit message: [cad & i2c] Figuring out I2C issues
Parts:
- added PULLDOWN, PULLDOWN_2: 12k, eagle-ltspice:R0207/10
Connections:
- new net N$1: LIDAR_LITE_V3.2, PULLDOWN_2.2
- new net N$2: LIDAR_LITE_V3.3, PULLDOWN.2
- net GND: now also PULLDOWN.1, PULLDOWN_2.1
Changed lines of the file:
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@@
 <layer number="97" name="Info" color="7" fill="1" visible="yes" active="yes"/>
 <layer number="98" name="Guide" color="6" fill="1" visible="yes" active="yes"/>
+<layer number="99" name="SpiceOrder" color="5" fill="1" visible="yes" active="yes"/>
 </layers>
 <schematic xreflabel="%F%N/%S.%C%R" xrefpart="/%S.%C%R">
@@
 <part name="SDA_PULLUP" library="rcl" deviceset="R-EU_" device="0204/2V" value="4.7k"/>
 <part name="SCL_PULLUP" library="rcl" deviceset="R-EU_" device="0204/2V" value="4.7k"/>
+<part name="PULLDOWN_2" library="eagle-ltspice" deviceset="R" device="0207/10" value="12k"/>
+<part name="PULLDOWN" library="eagle-ltspice" deviceset="R" device="0207/10" value="12k"/>
 </parts>
 <sheets>
@@
 <instance part="SDA_PULLUP" gate="G$1" x="76.2" y="99.06"/>
 <instance part="SCL_PULLUP" gate="G$1" x="73.66" y="106.68"/>
+<instance part="PULLDOWN_2" gate="G$1" x="83.82" y="149.86"/>
+<instance part="PULLDOWN" gate="G$1" x="76.2" y="142.24"/>
 </instances>
 <busses>
@@
 <pinref part="PAN_SERVO" gate="G$1" pin="3"/>
 <junction x="93.98" y="88.9"/>
+<pinref part="PULLDOWN_2" gate="G$1" pin="1"/>
+<wire x1="78.74" y1="149.86" x2="63.5" y2="149.86" width="0.1524" layer="91"/>
+<wire x1="63.5" y1="149.86" x2="63.5" y2="142.24" width="0.1524" layer="91"/>
+<junction x="63.5" y="137.16"/>
+<pinref part="PULLDOWN" gate="G$1" pin="1"/>
+<wire x1="63.5" y1="142.24" x2="63.5" y2="137.16" width="0.1524" layer="91"/>
+<wire x1="71.12" y1="142.24" x2="63.5" y2="142.24" width="0.1524" layer="91"/>
+<junction x="63.5" y="142.24"/>
+<label x="63.5" y="149.86" size="1.778" layer="95"/>
 </segment>
 </net>
@@
 </segment>
 </net>
+<net name="N$1" class="0">
+<segment>
+<pinref part="LIDAR_LITE_V3" gate="1" pin="2"/>
+<wire x1="93.98" y1="121.92" x2="93.98" y2="149.86" width="0.1524" layer="91"/>
+<pinref part="PULLDOWN_2" gate="G$1" pin="2"/>
+<wire x1="93.98" y1="149.86" x2="88.9" y2="149.86" width="0.1524" layer="91"/>
+</segment>
+</net>
+<net name="N$2" class="0">
+<segment>
+<pinref part="PULLDOWN" gate="G$1" pin="2"/>
+<wire x1="81.28" y1="142.24" x2="91.44" y2="142.24" width="0.1524" layer="91"/>
+<wire x1="91.44" y1="142.24" x2="91.44" y2="119.38" width="0.1524" layer="91"/>
+<pinref part="LIDAR_LITE_V3" gate="1" pin="3"/>
+<wire x1="91.44" y1="119.38" x2="93.98" y2="119.38" width="0.1524" layer="91"/>
+</segment>
+</net>
